Commit message: creacion de mapa

File: easybot_description/urdf/easybot_gazebo.xacro (robot description, xacro)
@@ -1,4 +1,5 @@
 <?xml version="1.0"?>
 <robot xmlns:xacro="http://ros.org/wiki/xacro">
+  <xacro:property name="PI" value="3.14159265"/>
     <gazebo>
         <plugin filename="libignition-gazebo-diff-drive-system.so" name="ignition::gazebo::systems::DiffDrive">
@@ -12,4 +13,5 @@
             <topic>cmd_vel</topic>
             <odom_topic>odom</odom_topic>
+            <tf_topic>/tf</tf_topic>
             <frame_id>odom</frame_id>
             <child_frame_id>base_link</child_frame_id>
@@ -21,22 +23,29 @@
     <gazebo reference="lidar_1">
         <sensor name="lidar_sensor" type="gpu_lidar">
-            <topic>scan</topic>
+            <ignition_frame_id>lidar_1</ignition_frame_id>
             <update_rate>10</update_rate>
-            <ignition_frame_id>lidar_1</ignition_frame_id>
-            <lidar>
+            <ray>
                 <scan>
                     <horizontal>
                         <samples>360</samples>
                         <resolution>1</resolution>
-                        <min_angle>-3.14159</min_angle>
-                        <max_angle>3.14159</max_angle>
+                        <min_angle>${-PI}</min_angle>
+                        <max_angle>${PI}</max_angle>
                     </horizontal>
                 </scan>
                 <range>
-                    <min>0.12</min> <max>10.0</max> <resolution>0.01</resolution>
+                    <min>0.12</min>
+                    <max>10.0</max>
+                    <resolution>0.017453</resolution>
                 </range>
-            </lidar>
+                <noise>
+                    <type>gaussian</type>
+                    <mean>0.0</mean>
+                    <stddev>0.01</stddev>
+                </noise>
+            </ray>
             <always_on>1</always_on>
             <visualize>true</visualize>
+            <topic>/scan</topic>
         </sensor>
     </gazebo>
